Commit message: Add files via upload

File: description/robot_core.xacro (robot description, xacro)
@@ -4,5 +4,5 @@
         <visual>
             <geometry>
-                <mesh filename="package://auto_tb/meshes/moborobo_short.stl" scale="1 1 1"/>
+                <mesh filename="package://moborobo/meshes/moborobo_short.stl" scale="1 1 1"/>
             </geometry>
         </visual>
